File: 8knobs_mono/8knobs.sch (KiCad schematic (older format))
At the start: 31 parts, among them J1 Conn_01x04_Female, U1 PC900, U2 BluePill_STM32F103C

Commit message: v1.1 of 8knobs mono:  - corrected wrong connection to battery  - easier PCB manufacturing
Connections:
- net at U2.1 (VBAT): no longer TP9.1
- net at U2.38 (5V_USB): now also TP9.1
Changed lines of the file:
@@
 NoConn ~ 9950 3950
 NoConn ~ 9950 4050
-NoConn ~ 8550 4900
 NoConn ~ 8250 4900
 NoConn ~ 8150 4900
@@
 	1    0    0    -1
 $EndComp
-Wire Wire Line
-	9500 2900 8750 2900
-Wire Wire Line
-	8750 2900 8750 3150
 $Comp
 L Connector:TestPoint TP10
@@
 NoConn ~ 8450 4900
 NoConn ~ 8350 3150
+NoConn ~ 8750 3150
+Wire Wire Line
+	10800 2900 10800 4900
+Wire Wire Line
+	9500 2900 10800 2900
+Wire Wire Line
+	10800 4900 9050 4900
+Wire Wire Line
+	9050 4900 9050 5200
+Wire Wire Line
+	9050 5200 8550 5200
+Wire Wire Line
+	8550 5200 8550 4900
 $EndSCHEMATC
